Commit message: Adapt paths.

File: robot_description/mild.urdf (robot description, URDF)
Before this commit: robot mild, 10 links, 9 joints
Links:
- link base_link: geometry visual mesh filename=package://asr_mild_kinematic_chain/robot_description/mild.d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
- link ptu_mount_link: geometry visual mesh filename=package://asr_mild_kinematic_chain/robot_description/camera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

Commit message: Adapt TF for NBV.

File: robot_description/mild.urdf (robot description, URDF)
Before this commit: robot mild, 10 links, 9 joints
Joints:
- joint base_to_ptu: origin xyz=0.0 -0.03 1.425 -> xyz=0.0 0.0 1.425
